File: thermal-flashlight.brd (EAGLE design)
At the start: 49.5 x 37.1 mm, 28 parts, among them IC1 ATMEGA328P, IC2 MCP73831, IC4 MCP1700-33, J1 AYZ0202, Q4 BSS123, U1 MLX90614_, X1 USBSMD

Commit message: update
Parts:
- added SV1: (no value), con-lstb:MA05-2
Connections:
- new net N$12: IC1.19
- new net N$13: IC1.22
- net A0: now also SV1.4
- net A1: now also SV1.2
- net A2: now also SV1.9
- net D3: now also SV1.10
- net D5: now also SV1.8
- net D6: now also SV1.6
- net GND: now also SV1.1
- net SCL: now also SV1.5
- net SDA: now also SV1.7
- net VCC: now also SV1.3
Routing:
- net GND: track 0.00 -> 145.2 mm
- net VBAT: track 0.00 -> 129.1 mm
- net VCC: track 0.00 -> 126.9 mm, vias 0 -> 3
- net A2: track 0.00 -> 76.2 mm, vias 0 -> 1
- net VBUS: track 0.00 -> 76.1 mm, vias 0 -> 3
- net SDA: track 0.00 -> 71.2 mm, vias 0 -> 1
- net D3: track 0.00 -> 70.8 mm, vias 0 -> 1
- net VDD: track 0.00 -> 58.0 mm, vias 0 -> 3
- net SCL: track 0.00 -> 54.7 mm, vias 0 -> 1
- net A0: track 0.00 -> 50.9 mm, vias 0 -> 1
- net RESET: track 0.00 -> 47.9 mm, vias 0 -> 1
- net A1: track 0.00 -> 46.1 mm, vias 0 -> 1
- net D5: track 0.00 -> 41.7 mm, vias 0 -> 2
- net D6: track 0.00 -> 41.0 mm, vias 0 -> 2
- net D4: track 0.00 -> 35.6 mm, vias 0 -> 2
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Other:
- board size 49.5 x 37.1 mm -> 49.5 x 38.4 mm
- board text added: "A0"
- board text added: "A1"
- board text added: "A2"
- board text added: "D3"
- board text added: "D5"
- board text added: "D6"
- board text added: "GND"
- board text added: "SCL"
- board text added: "SDA"
- board text added: "VCC"
