File: thermal-flashlight.brd (EAGLE design)
At the start: 49.5 x 38.4 mm, 29 parts, among them IC1 ATMEGA328P, IC2 MCP73831, IC4 MCP1700-33, J1 AYZ0202, Q4 BSS123, U1 MLX90614_, X1 USBSMD

Commit message: update
Other:
- board size 49.5 x 38.4 mm -> 49.5 x 42.9 mm
Changed lines of the file:
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@@
 <setting verticaltext="up"/>
 </settings>
-<grid distance="0.01" unitdist="inch" unit="inch" style="lines" multiple="1" display="yes" altdistance="0.01" altunitdist="inch" altunit="inch"/>
+<grid distance="0.05" unitdist="inch" unit="inch" style="lines" multiple="1" display="yes" altdistance="0.01" altunitdist="inch" altunit="inch"/>
 <layers>
 <layer number="1" name="Top" color="4" fill="1" visible="yes" active="yes"/>
@@
 <layer number="43" name="vRestrict" color="2" fill="10" visible="yes" active="yes"/>
 <layer number="44" name="Drills" color="7" fill="1" visible="no" active="yes"/>
-<layer number="45" name="Holes" color="7" fill="1" visible="no" active="yes"/>
+<layer number="45" name="Holes" color="7" fill="1" visible="yes" active="yes"/>
 <layer number="46" name="Milling" color="3" fill="1" visible="no" active="yes"/>
 <layer number="47" name="Measures" color="7" fill="1" visible="no" active="yes"/>
@@
 <plain>
 <wire x1="2.54" y1="0" x2="41.91" y2="0" width="0" layer="20"/>
-<wire x1="49.53" y1="2.54" x2="49.53" y2="38.354" width="0" layer="20"/>
-<wire x1="49.53" y1="38.354" x2="0" y2="38.354" width="0" layer="20"/>
-<wire x1="0" y1="38.354" x2="0" y2="2.54" width="0" layer="20"/>
+<wire x1="49.53" y1="2.54" x2="49.53" y2="42.926" width="0" layer="20"/>
+<wire x1="49.53" y1="42.926" x2="0" y2="42.926" width="0" layer="20"/>
+<wire x1="0" y1="42.926" x2="0" y2="2.54" width="0" layer="20"/>
 <wire x1="0" y1="2.54" x2="2.54" y2="0" width="0" layer="20" curve="90"/>
 <text x="2.032" y="23.368" size="1.016" layer="25" ratio="20" rot="R90">On</text>
@@
 <text x="10.414" y="34.544" size="1.016" layer="25" ratio="20" rot="R180">FLASHLIGHT!</text>
 <text x="12.192" y="37.592" size="1.016" layer="25" ratio="20" rot="R180">PUBLICLAB.ORG</text>
+<hole x="5.08" y="40.132" drill="2.2"/>
+<hole x="11.43" y="40.132" drill="2.2"/>
+<hole x="17.78" y="40.132" drill="2.2"/>
+<hole x="24.13" y="40.132" drill="2.2"/>
+<hole x="30.48" y="40.132" drill="2.2"/>
+<hole x="36.83" y="40.132" drill="2.2"/>
+<hole x="43.18" y="40.132" drill="2.2"/>
 </plain>
 <attributes>

Commit message: update
Parts:
- moved J1 3.82 mm to (4.32, 32.3)
- moved RIR1 3.82 mm to (9.40, 32.3)
- moved U$1 3.82 mm to (26.4, 29.2)
- moved RIR2 3.82 mm to (22.9, 35.8)
- moved C5 3.82 mm to (18.5, 19.6)
- moved IC1 3.82 mm to (17.5, 13.0)
- moved IC4 3.82 mm to (28.4, 11.9)
- moved RD+ 3.82 mm to (14.0, 19.6)
- moved RN1 3.82 mm to (24.9, 11.9)
- moved C1 3.82 mm to (34.5, 6.60)
- moved C2 3.82 mm to (32.3, 6.60)
- moved C4 3.82 mm to (15.7, 6.10)
- moved RC 3.82 mm to (29.7, 6.60)
- moved RRST 3.82 mm to (12.2, 7.11)
- moved X 3.82 mm to (19.8, 6.10)
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Routing:
- net GND: track 145.2 -> 0.00 mm
- net VBAT: track 129.1 -> 0.00 mm
- net VCC: track 126.9 -> 0.00 mm, vias 3 -> 0
- net A2: track 76.2 -> 0.00 mm, vias 1 -> 0
- net VBUS: track 76.1 -> 0.00 mm, vias 3 -> 0
- net SDA: track 71.2 -> 0.00 mm, vias 1 -> 0
- net D3: track 70.8 -> 0.00 mm, vias 1 -> 0
- net VDD: track 58.0 -> 0.00 mm, vias 3 -> 0
- net SCL: track 54.7 -> 0.00 mm, vias 1 -> 0
- net A0: track 50.9 -> 0.00 mm, vias 1 -> 0
- net RESET: track 47.9 -> 0.00 mm, vias 1 -> 0
- net A1: track 46.1 -> 0.00 mm, vias 1 -> 0
- net D5: track 41.7 -> 0.00 mm, vias 2 -> 0
- net D6: track 41.0 -> 0.00 mm, vias 2 -> 0
- net D4: track 35.6 -> 0.00 mm, vias 2 -> 0
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Other:
- board size 49.5 x 42.9 mm -> 49.8 x 42.9 mm
- board text added: "PUBLICLAB.org"
- board text added: "THERMAL-FLASHLIGHT"
- board text added: "http://publiclab.org/wiki/thermal-flashlight"
- board text removed: "FLASHLIGHT!"
- board text removed: "PUBLICLAB.ORG"
- board text removed: "THERMAL"
- board text removed: "publiclab.org/wiki/thermal-flashlight"

Commit message: update
Routing:
- net GND: track 0.00 -> 145.4 mm, vias 0 -> 2
- net VCC: track 0.00 -> 112.8 mm, vias 0 -> 2
- net VBUS: track 0.00 -> 90.2 mm, vias 0 -> 3
- net VBAT: track 0.00 -> 72.8 mm, vias 0 -> 2
- net D3: track 0.00 -> 67.7 mm, vias 0 -> 1
- net VDD: track 0.00 -> 66.9 mm, vias 0 -> 4
- net SCL: track 0.00 -> 63.4 mm
- net SDA: track 0.00 -> 61.4 mm, vias 0 -> 2
- net A2: track 0.00 -> 61.2 mm, vias 0 -> 1
- net D5: track 0.00 -> 60.3 mm
- net RESET: track 0.00 -> 52.0 mm, vias 0 -> 3
- net MISO: track 0.00 -> 43.7 mm, vias 0 -> 1
- net D6: track 0.00 -> 38.2 mm, vias 0 -> 1
- net SCK: track 0.00 -> 36.9 mm, vias 0 -> 2
- net D4: track 0.00 -> 35.4 mm, vias 0 -> 2
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