File: thermal-flashlight-32u4-many.sch (EAGLE design)
At the start: 36 parts, among them IC2 MCP73831, IC3 ATMEGA32U4-AU, IC4 MCP1700-33, J1 AYZ0202, J2 1X2-3.5MM, Q4 BSS123, U1 MLX90614_, X1 USBSMD, X3 8MHz

Commit message: update
Connections:
- net A2: no longer SV1.6
- net A3: no longer SV1.5
- net D0/RX: now also SV1.6
- net D1/TX: now also SV1.5
Changed lines of the file:
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@@
 <setting verticaltext="up"/>
 </settings>
-<grid distance="0.01" unitdist="inch" unit="inch" style="lines" multiple="1" display="no" altdistance="0.01" altunitdist="inch" altunit="inch"/>
+<grid distance="0.1" unitdist="inch" unit="inch" style="lines" multiple="1" display="no" altdistance="0.01" altunitdist="inch" altunit="inch"/>
 <layers>
 <layer number="1" name="Top" color="4" fill="1" visible="no" active="no"/>
@@
 <label x="71.374" y="49.784" size="1.778" layer="95"/>
 </segment>
-<segment>
-<pinref part="SV1" gate="1" pin="6"/>
-<wire x1="120.142" y1="-11.43" x2="117.856" y2="-11.43" width="0.1524" layer="91"/>
-<label x="113.792" y="-11.43" size="1.778" layer="95"/>
-</segment>
 </net>
 <net name="A3" class="0">
@@
 <wire x1="70.866" y1="52.07" x2="70.866" y2="52.324" width="0.1524" layer="91"/>
 <label x="71.12" y="52.578" size="1.778" layer="95"/>
-</segment>
-<segment>
-<pinref part="SV1" gate="1" pin="5"/>
-<wire x1="135.382" y1="-11.43" x2="137.668" y2="-11.43" width="0.1524" layer="91"/>
-<label x="138.176" y="-10.922" size="1.778" layer="95"/>
 </segment>
 </net>
@@
 <pinref part="IC3" gate="G$1" pin="PD3(INT3/TXD1)"/>
 </segment>
+<segment>
+<pinref part="SV1" gate="1" pin="5"/>
+<wire x1="135.382" y1="-11.43" x2="137.668" y2="-11.43" width="0.1524" layer="91"/>
+<label x="138.176" y="-10.922" size="1.778" layer="95"/>
+</segment>
 </net>
 <net name="D0/RX" class="0">
@@
 <pinref part="IC3" gate="G$1" pin="PD2(INT2/RXD1)"/>
 </segment>
-</net>
+<segment>
+<pinref part="SV1" gate="1" pin="6"/>
+<wire x1="120.142" y1="-11.43" x2="117.856" y2="-11.43" width="0.1524" layer="91"/>
+<label x="109.474" y="-11.43" size="1.778" layer="95"/>
+</segment>
+</net>
