File: thermal-flashlight-32u4-many.brd (EAGLE design)
At the start: 49.8 x 46.2 mm, 36 parts, among them IC2 MCP73831, IC3 ATMEGA32U4-AU, IC4 MCP1700-33, J1 AYZ0202, J2 1X2-3.5MM, Q4 BSS123, U1 MLX90614_, X1 USBSMD, X3 8MHz

Commit message: update
Parts:
- removed C6, C7: 18pF, adafruit:C0805K
- removed X3: 8MHz, adaprog:NX5032
- added X2: 12MHz, SparkFunNew:RESONATOR-SMD
- moved C1 12.0 mm to (12.4, 3.56), turned to 0 degrees
- moved C2 4.38 mm to (22.6, 3.56), turned to 0 degrees
- moved RIR1 1.80 mm to (31.0, 21.8)
- moved IC4 1.78 mm to (29.5, 17.5)
- moved Q4 1.78 mm to (29.5, 13.0)
- moved IC2 1.70 mm to (28.7, 4.06)
- moved C3 1.55 mm to (29.0, 8.64)
- moved RIR2 1.52 mm to (27.9, 21.8)
- moved IC3 1.05 mm to (19.3, 13.2)
- moved SV1 0.92 mm to (21.3, 24.9)
- moved CHG 0.92 mm to (7.62, 3.56)
- moved U$1 0.80 mm to (31.2, 31.2)
- moved RC 0.57 mm to (34.0, 3.30)
- moved RN3 0.51 mm to (33.3, 42.9)
- moved RN4 0.51 mm to (43.9, 42.9)
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Connections:
- removed net N$15: C7.1, IC3.16, X3.P$1
- removed net N$16: C6.1, IC3.17, X3.P$2
- new net N$22: X2.1
- new net N$23: X2.3
- net GND: now also X2.2; no longer C6.2, C7.2
Other:
- outline, holes or cut-outs redrawn

Commit message: update
Parts:
- removed X2: 12MHz, SparkFunNew:RESONATOR-SMD
- added C6, C7: 18pF, adafruit:C0805K
- added X3: 8MHz, adaprog:NX5032
- moved C1 12.0 mm to (24.4, 4.32), turned to 90 degrees
- moved C2 4.38 mm to (26.9, 4.32), turned to 90 degrees
- moved RIR1 1.80 mm to (31.2, 23.6)
- moved IC4 1.78 mm to (29.5, 19.3)
- moved Q4 1.78 mm to (29.5, 14.7)
- moved IC2 1.70 mm to (30.2, 4.83)
- moved C3 1.55 mm to (29.2, 10.2)
- moved RIR2 1.52 mm to (27.9, 23.4)
- moved IC3 1.05 mm to (19.1, 14.2)
- moved SV1 0.92 mm to (21.8, 25.7)
- moved CHG 0.92 mm to (6.86, 4.06)
- moved U$1 0.80 mm to (31.5, 32.0)
- moved RC 0.57 mm to (34.5, 3.56)
- moved BAT1 0.51 mm to (41.4, 25.7)
- moved LED 0.25 mm to (7.62, 42.9)
Connections:
- removed net N$22: X2.1
- removed net N$23: X2.3
- new net N$15: C7.1, IC3.16, X3.P$1
- new net N$16: C6.1, IC3.17, X3.P$2
- net GND: now also C6.2, C7.2; no longer X2.2

Commit message: update
Parts:
- moved RIR2 3.57 mm to (31.5, 23.6)
- moved RIR1 3.30 mm to (27.9, 23.6)
- moved J2 1.05 mm to (45.2, 32.0)
- moved RTHERM 0.36 mm to (38.6, 31.8)
- moved BTN 0.25 mm to (12.2, 34.0)
- moved U1 0.25 mm to (20.8, 34.5)
Connections:
- net A2: no longer SV1.6
- net A3: no longer SV1.5
- net D0/RX: now also SV1.6
- net D1/TX: now also SV1.5
Routing:
- net SCK: track 0.00 -> 127.3 mm, vias 0 -> 3
- net VCC: track 0.00 -> 119.7 mm
- net MISO: track 0.00 -> 113.4 mm, vias 0 -> 3
- net VBAT: track 0.00 -> 92.2 mm
- net VBUS: track 0.00 -> 92.0 mm, vias 0 -> 4
- net D8: track 0.00 -> 87.8 mm, vias 0 -> 2
- net VDD: track 0.00 -> 75.6 mm, vias 0 -> 3
- net SDA: track 0.00 -> 52.4 mm, vias 0 -> 1
- net N$10: track 0.00 -> 46.3 mm, vias 0 -> 2
- net SCL: track 0.00 -> 46.0 mm, vias 0 -> 1
- net A4: track 0.00 -> 40.4 mm, vias 0 -> 1
- net MOSI: track 0.00 -> 33.7 mm, vias 0 -> 2
- net RST: track 0.00 -> 31.4 mm, vias 0 -> 2
- net GND: track 0.00 -> 27.7 mm
- net N$5: track 0.00 -> 27.2 mm, vias 0 -> 2
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- added copper zone on layer 1, net GND
Other:
- board size 49.8 x 46.2 mm -> 49.3 x 46.2 mm
- board text added: "PUBLICLAB.ORG"
- board text added: "RX"
- board text added: "THERMAL*FLASHLIGHT"
- board text added: "TX"
- board text removed: "*THERMAL*FLASHLIGHT*"
- board text removed: "A2"
- board text removed: "A3"
